File: garden36.kicad_pcb (KiCad board)
At the start: 2 copper layers, 231.5 x 91.8 mm, 96 parts, among them J1 Conn_01x02, J2 Conn_01x02, SW1 SW_SPDT, SW2 SW_Push, SW3 SW_SPDT, SW4 SW_Push, U1 nice_nano, U2 nice_nano

Commit message: V2 started
Parts:
- removed the REF** at (237.4, 71.1)
- removed the REF** at (111.7, 64.3)
- removed the REF** at (46.7, 124.6)
- removed the REF** at (121.9, 106.6)
- removed the REF** at (154.6, 106.6)
- removed the REF** at (39.2, 71.1)
- removed the REF** at (164.9, 64.3)
- removed the REF** at (119.9, 133.8)
- removed the REF** at (156.7, 133.8)
- removed the REF** at (229.9, 124.6)
- CH19, CH20, CH21, CH22, CH23, CH24, CH25, CH26, CH27, CH28, CH29, CH30, CH31, CH32, CH33, CH34, CH35, CH36, D19, D20, D21, D22, D23, D24, D25, D26, D27, D28, D29, D30, D31, D32, D33, D34, D35, D36: moved to F.Cu
- SW1: moved to B.Cu
- moved CH21 268.5 mm to (44.6, -63.8), turned to 0 degrees
- moved CH20 268.1 mm to (44.6, -80.2), turned to 0 degrees
- moved CH19 267.7 mm to (44.6, -96.5), turned to 0 degrees
- moved CH32 230.6 mm to (79.8, -80.2), turned to 0 degrees
- moved D21 227.4 mm to (92.7, -58.6)
- moved CH31 226.3 mm to (79.8, -96.5), turned to 0 degrees
- moved D20 217.4 mm to (92.7, -61.9)
- moved CH28 216.3 mm to (62.2, -47.5), turned to 0 degrees
- moved CH24 216.2 mm to (44.6, -14.8), turned to 0 degrees
- moved CH23 215.9 mm to (44.6, -31.1), turned to 0 degrees
- moved CH22 215.5 mm to (44.6, -47.5), turned to 0 degrees
- moved CH27 215.2 mm to (62.2, -63.8), turned to 0 degrees
- moved CH26 214.8 mm to (62.2, -80.2), turned to 0 degrees
- moved CH25 214.3 mm to (62.2, -96.5), turned to 0 degrees
- moved D19 207.8 mm to (92.7, -65.3)
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Connections:
- net +3.3Vx renamed R_+3.3V
- net CSx renamed R_CS
- net RSTx renamed R_RST
- CH19 pad 1: COL5 -> R_COL0
- CH20 pad 1: COL5 -> R_COL1
- CH21 pad 1: COL5 -> R_COL2
- CH22 pad 1: COL6 -> R_COL3
- CH23 pad 1: COL6 -> R_COL4
- CH24 pad 1: COL6 -> R_COL0
- CH25 pad 1: COL7 -> R_COL1
- CH26 pad 1: COL7 -> R_COL2
- CH27 pad 1: COL7 -> R_COL3
- CH28 pad 1: COL7 -> R_COL4
- CH29 pad 1: COL8 -> R_COL0
- CH30 pad 1: COL8 -> R_COL1
- CH31 pad 1: COL8 -> R_COL2
- CH32 pad 1: COL8 -> R_COL3
- CH33 pad 1: COL9 -> R_COL4
- CH34 pad 1: COL9 -> R_COL0
- CH35 pad 1: COL9 -> R_COL1
- CH36 pad 1: COL9 -> R_COL2
- D19 pad 1: ROW4 -> R_ROW0
- D20 pad 1: ROW5 -> R_ROW0
- D21 pad 1: ROW6 -> R_ROW0
- D22 pad 1: ROW4 -> R_ROW0
- D23 pad 1: ROW5 -> R_ROW0
- D24 pad 1: ROW6 -> R_ROW1
- D25 pad 1: ROW4 -> R_ROW1
- D26 pad 1: ROW5 -> R_ROW1
- D27 pad 1: ROW6 -> R_ROW1
- D28 pad 1: ROW7 -> R_ROW1
- D29 pad 1: ROW4 -> R_ROW2
- D30 pad 1: ROW5 -> R_ROW2
- D31 pad 1: ROW6 -> R_ROW2
- D32 pad 1: ROW7 -> R_ROW2
- D33 pad 1: ROW4 -> R_ROW2
- D34 pad 1: ROW5 -> R_ROW3
- D35 pad 1: ROW6 -> R_ROW3
- D36 pad 1: ROW7 -> R_ROW3
- Display2 pad 1: MOSIx -> R_MOSI
- Display2 pad 2: SCKx -> R_SCK
- Display2 pad 4: GNDx -> R_GND
- J2 pad 1: BATx -> R_BAT
- J2 pad 2: GNDx -> R_GND
- SW1 pad 3: BAT -> RAW
- SW3 pad 2: BATx -> R_BAT
- SW3 pad 3: BATx -> R_RAW
- SW4 pad 2: GNDx -> R_GND
- U1 pad 12: ROW3 -> unconnected-(U1-P1.06-LF-Pad12)
- U1 pad 13: BAT -> RAW
- U1 pad 17: COL0 -> unconnected-(U1-P0.31-LF-Pad17)
- U1 pad 18: COL1 -> unconnected-(U1-P0.29-LF-Pad18)
- U1 pad 19: COL2 -> unconnected-(U1-P0.02-LF-Pad19)
- U1 pad 20: COL3 -> unconnected-(U1-P1.15-LF-Pad20)
- U1 pad 21: COL4 -> unconnected-(U1-P1.13-LF-Pad21)
- U1 pad 28: GND -> B-
- U1 pad 29: BAT -> B+
- U1 pad 5: SCK -> MOSI
- U1 pad 6: MOSI -> SCK
- U1 pad 7: ROW0 -> unconnected-(U1-P0.22-Pad7)
- U1 pad 8: ROW1 -> unconnected-(U1-P0.24-Pad8)
- U1 pad 9: ROW2 -> unconnected-(U1-P1.00-Pad9)
- U2 pad 10: COL8 -> unconnected-(U2-P0.11-Pad10)
- U2 pad 11: COL9 -> unconnected-(U2-P1.04-LF-Pad11)
- U2 pad 13: BATx -> R_RAW
- U2 pad 14: GNDx -> R_GND
- U2 pad 21: ROW4 -> unconnected-(U2-P1.13-LF-Pad21)
- U2 pad 22: ROW5 -> unconnected-(U2-P1.11-LF-Pad22)
- U2 pad 23: ROW6 -> unconnected-(U2-P0.10-LF-Pad23)
- U2 pad 24: ROW7 -> unconnected-(U2-P0.09-LF-Pad24)
- U2 pad 28: GNDx -> R_B-
- U2 pad 29: BATx -> R_B+
- U2 pad 3: GNDx -> R_GND
- U2 pad 4: GNDx -> R_GND
- U2 pad 5: SCKx -> R_MOSI
- U2 pad 6: MOSIx -> R_SCK
- U2 pad 7: COL5 -> unconnected-(U2-P0.22-Pad7)
- U2 pad 8: COL6 -> unconnected-(U2-P0.24-Pad8)
- U2 pad 9: COL7 -> unconnected-(U2-P1.00-Pad9)
Routing:
- net COL5: track 147.3 -> 0.00 mm
- net COL7: track 142.2 -> 0.00 mm
- net ROW6: track 135.1 -> 0.00 mm
- net COL8: track 129.9 -> 0.00 mm
- net COL6: track 123.8 -> 0.00 mm
- net ROW4: track 122.9 -> 0.00 mm
- net ROW5: track 118.9 -> 0.00 mm
- net COL0: track 139.2 -> 36.7 mm
- net GNDx: track 101.9 -> 0.00 mm
- net GND: track 89.5 -> 0.00 mm
- net COL1: track 117.4 -> 36.8 mm
- net ROW7: track 79.7 -> 0.00 mm
- net BATx: track 78.6 -> 0.00 mm
- net COL9: track 69.1 -> 0.00 mm
- net COL2: track 144.1 -> 77.3 mm
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- added copper zone on F.Cu, net COL0

Commit message: Update libraries continue with updates for project
Parts:
- removed J1, J2: Conn_01x02, Connector_JST:JST_PH_S2B-PH-K_1x02_P2.00mm_Horizontal
- removed REF** (x2): mousebites 1mm, PCM_marbastlib-various:mousebites_1mm
- CH19, CH20, CH21, CH22, CH23, CH24, CH25, CH26, CH27, CH28, CH29, CH30, CH31, CH32, CH33, CH34, CH35, CH36, D19, D20, D21, D22, D23, D24, D25, D26, D27, D28, D29, D30, D31, D32, D33, D34, D35, D36: moved to B.Cu
- SW2, SW4: footprint Button_Switch_SMD:SW_SPST_TL3305A -> Button_Switch_SMD:SW_SPST_B3U-1000P
- moved CH31 240.3 mm to (205.0, 108.5)
- moved CH32 236.6 mm to (223.2, 107.9)
- moved CH33 233.7 mm to (239.0, 107.2)
- moved CH25 227.1 mm to (188.0, 92.5)
- moved CH28 224.7 mm to (238.5, 91.8)
- moved CH26 223.8 mm to (205.2, 91.9)
- moved CH27 223.4 mm to (222.5, 91.8)
- moved CH23 220.5 mm to (237.9, 74.8)
- moved D33 219.1 mm to (233.8, 111.5)
- moved CH22 214.6 mm to (221.2, 74.2)
- moved CH19 213.8 mm to (172.2, 75.0)
- moved CH20 212.0 mm to (189.2, 74.8)
- moved CH21 211.5 mm to (204.5, 74.5)
- moved D28 205.1 mm to (233.8, 95.5)
- moved D36 203.0 mm to (188.0, 129.8)
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Connections:
- U1 pad 28: B- -> unconnected-(U1-GND-Pad28)
- U1 pad 29: B+ -> unconnected-(U1-BAT+-Pad29)
- U2 pad 28: R_B- -> unconnected-(U2-GND-Pad28)
- U2 pad 29: R_B+ -> unconnected-(U2-BAT+-Pad29)
Other:
- board text added: "v1.1"
- board text removed: "v1.0"

Commit message: Switches set
Parts:
- added PW1: ~, garden:Battery, F.Cu at (125.8, 101.8)
- added PW4: ~, garden:Battery, F.Cu at (150.7, 101.8)
- added REF**: mousebites 1mm, PCM_marbastlib-various:mousebites_1mm, F.Cu at (140.8, 99.3)
- added REF**: mousebites 1mm, PCM_marbastlib-various:mousebites_1mm, B.Cu at (135.8, 99.3)
- SW2, SW3, SW4: moved to B.Cu
- moved SW1 75.8 mm to (109.4, 58.0)
- moved SW4 43.5 mm to (177.1, 58.8), turned to -90 degrees
- moved SW3 39.4 mm to (167.1, 58.0), turned to 180 degrees
- moved D31 18.8 mm to (207.3, 99.2), turned to 180 degrees
- moved CH26 14.5 mm to (207.9, 77.6)
- moved D21 14.4 mm to (207.8, 65.2), turned to 180 degrees
- moved D26 14.3 mm to (207.8, 82.2), turned to 180 degrees
- moved CH21 14.3 mm to (207.9, 60.6)
- moved CH31 14.2 mm to (207.9, 94.6)
- moved D33 13.5 mm to (243.8, 120.7), turned to 180 degrees
- moved D28 12.9 mm to (243.8, 103.7), turned to 180 degrees
- moved D30 10.6 mm to (189.8, 105.7), turned to 180 degrees
- moved CH33 10.1 mm to (243.9, 116.1)
- moved D23 9.76 mm to (243.8, 86.7), turned to 180 degrees
- moved CH23 9.44 mm to (243.9, 82.1)
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Connections:
- SW1 pad 2: BAT -> Net-(PW1-BAT+)
- SW3 pad 2: R_BAT -> Net-(PW4-BAT+)
Routing:
- net ROW0: track 89.2 -> 0.00 mm
- net ROW2: track 88.5 -> 0.00 mm
- net ROW1: track 88.5 -> 0.00 mm
- net COL3: track 78.1 -> 0.00 mm
- net COL2: track 77.3 -> 0.00 mm
- net COL4: track 60.6 -> 0.00 mm
- net ROW3: track 42.7 -> 0.00 mm
- net BAT: track 40.5 -> 0.00 mm, vias 1 -> 0
- net COL1: track 36.8 -> 0.00 mm
- net COL0: track 36.7 -> 0.00 mm
- net Net-(D18-A): track 11.5 -> 0.00 mm
- net Net-(D17-A): track 11.4 -> 0.00 mm
- net Net-(D7-A): track 11.2 -> 0.00 mm
- net Net-(D2-A): track 11.2 -> 0.00 mm
- net Net-(D12-A): track 11.2 -> 0.00 mm
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- removed copper zone on B.Cu, net (none)
- removed copper zone on F.Cu, net (none)
- removed copper zone on F.Cu, net COL0
Other:
- outline, holes or cut-outs redrawn
