File: garden36.kicad_sch (KiCad schematic)
At the start: 98 parts, among them SW1 SW_SPDT, SW2 SW_Push, SW3 SW_SPDT, SW4 SW_Push, U1 nice_nano, U2 nice_nano

Commit message: Finish design
Parts:
- removed PW1, PW4: ~, garden:Battery, symbol kometa:Battery
- added PW1, PW2: ~, garden:Battery, symbol garden:Battery
Connections:
- net COL0: now also U1.2 (P0.08)
- net COL1: now also U1.17 (P0.31-LF)
- net COL2: now also U1.18 (P0.29-LF)
- net COL3: now also U1.19 (P0.02-LF)
- net COL4: now also U1.20 (P1.15-LF)
- net GND: now also PW1.2 (BAT-)
- net RAW: now also U1.29 (BAT+)
- net ROW0: now also U1.21 (P1.13-LF)
- net ROW1: now also U1.22 (P1.11-LF)
- net ROW2: now also U1.23 (P0.10-LF)
- net ROW3: now also U1.24 (P0.09-LF)
- net R_COL0: now also U2.8 (P0.24)
- net R_COL1: now also U2.7 (P0.22)
- net R_COL2: now also U2.19 (P0.02-LF)
- net R_COL3: now also U2.18 (P0.29-LF)
- net R_COL4: now also U2.17 (P0.31-LF)
- net R_GND: now also PW2.2 (BAT-)
- net R_RAW: now also U2.29 (BAT+)
- net R_ROW0: now also U2.9 (P1.00)
- net R_ROW1: now also U2.10 (P0.11)
- net R_ROW2: now also U2.11 (P1.04-LF)
- net R_ROW3: now also U2.12 (P1.06-LF)
- net at SW1.2 (B): now also PW1.1 (BAT+)
- net at SW3.2 (B): now also PW2.1 (BAT+)
- no-connect marks 6 -> 22
Other:
- moved on the sheet: H11, H12, H13, H14, H15, H16, H17
